File: pcb/debug.kicad_sch (KiCad schematic)
At the start: 29 parts, among them J2 USB_C_Receptacle_USB2.0, SW1 SW_DIP_x02, U2 FT4222HQ, Y1 12MHz

Commit message: route the power supply
Parts:
- added D3: MMBZxx, Package_TO_SOT_SMD:SOT-23, symbol Diode:MMBZxx
Connections:
- net DP: now also D3.1 (K)
- net GND: now also D3.3 (A)
- net DM renamed DN
- net DN: now also D3.2 (K)
Changed lines of the file:
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@@
   (junction (at 163.83 120.65) (diameter 0) (color 0 0 0 0)
   )
+  (junction (at 120.65 90.17) (diameter 0) (color 0 0 0 0)
+  )
   (junction (at 161.29 139.7) (diameter 0) (color 0 0 0 0)
   )
@@
   )
   (junction (at 121.92 45.72) (diameter 0) (color 0 0 0 0)
+  )
+  (junction (at 125.73 87.63) (diameter 0) (color 0 0 0 0)
   )
   (junction (at 163.83 46.99) (diameter 0) (color 0 0 0 0)
@@
     (stroke (width 0) (type default) (color 0 0 0 0))
   )
+  (wire (pts (xy 125.73 87.63) (xy 173.99 87.63))
+    (stroke (width 0) (type default) (color 0 0 0 0))
+  )
   (wire (pts (xy 163.83 119.38) (xy 173.99 119.38))
     (stroke (width 0) (type default) (color 0 0 0 0))
@@
     (stroke (width 0) (type default) (color 0 0 0 0))
   )
+  (wire (pts (xy 120.65 90.17) (xy 173.99 90.17))
+    (stroke (width 0) (type default) (color 0 0 0 0))
+  )
+  (wire (pts (xy 125.73 87.63) (xy 125.73 92.71))
+    (stroke (width 0) (type default) (color 0 0 0 0))
+  )
+  (wire (pts (xy 91.44 92.71) (xy 92.71 92.71))
+    (stroke (width 0) (type default) (color 0 0 0 0))
+  )
   (wire (pts (xy 96.52 109.22) (xy 96.52 140.97))
     (stroke (width 0) (type default) (color 0 0 0 0))
@@
     (stroke (width 0) (type default) (color 0 0 0 0))
   )
-  (wire (pts (xy 91.44 92.71) (xy 92.71 92.71))
-    (stroke (width 0) (type default) (color 0 0 0 0))
-  )
   (wire (pts (xy 194.31 124.46) (xy 194.31 125.73))
     (stroke (width 0) (type default) (color 0 0 0 0))
@@
     (stroke (width 0) (type default) (color 0 0 0 0))
   )
-  (wire (pts (xy 92.71 87.63) (xy 173.99 87.63))
+  (wire (pts (xy 92.71 87.63) (xy 125.73 87.63))
     (stroke (width 0) (type default) (color 0 0 0 0))
   )
@@
     (stroke (width 0) (type default) (color 0 0 0 0))
   )
+  (wire (pts (xy 91.44 87.63) (xy 92.71 87.63))
+    (stroke (width 0) (type default) (color 0 0 0 0))
+  )
   (wire (pts (xy 215.9 54.61) (xy 224.79 54.61))
     (stroke (width 0) (type default) (color 0 0 0 0))
@@
     (stroke (width 0) (type default) (color 0 0 0 0))
   )
-  (wire (pts (xy 91.44 87.63) (xy 92.71 87.63))
-    (stroke (width 0) (type default) (color 0 0 0 0))
-  )
   (wire (pts (xy 104.14 109.22) (xy 104.14 140.97))
     (stroke (width 0) (type default) (color 0 0 0 0))
@@
     (stroke (width 0) (type default) (color 0 0 0 0))
   )
-  (wire (pts (xy 92.71 90.17) (xy 173.99 90.17))
+  (wire (pts (xy 92.71 90.17) (xy 120.65 90.17))
+    (stroke (width 0) (type default) (color 0 0 0 0))
+  )
+  (wire (pts (xy 123.19 102.87) (xy 123.19 140.97))
     (stroke (width 0) (type default) (color 0 0 0 0))
   )
@@
   )
   (wire (pts (xy 156.21 113.03) (xy 173.99 113.03))
+    (stroke (width 0) (type default) (color 0 0 0 0))
+  )
+  (wire (pts (xy 120.65 90.17) (xy 120.65 92.71))
     (stroke (width 0) (type default) (color 0 0 0 0))
   )
@@
     (effects (font (size 1.27 1.27)) (justify right bottom))
   )
-  (label "DM" (at 173.99 87.63 180)
+  (label "DN" (at 173.99 87.63 180)
     (effects (font (size 1.27 1.27)) (justify right bottom))
   )
@@
     (pin "1")
   )
+  (symbol (lib_id "Diode:MMBZxx") (at 123.19 97.79 0) (unit 1)
+    (in_bom yes) (on_board yes) (fields_autoplaced)
+    (property "Reference" "D3" (id 0) (at 128.27 96.6469 0)
+      (effects (font (size 1.27 1.27)) (justify left))
+    )
+    (property "Value" "MMBZxx" (id 1) (at 128.27 99.1869 0)
+      (effects (font (size 1.27 1.27)) (justify left))
+    )
+    (property "Footprint" "Package_TO_SOT_SMD:SOT-23" (id 2) (at 127 100.33 0)
+      (effects (font (size 1.27 1.27)) (justify left) hide)
+    )
+    (property "Datasheet" "http://www.onsemi.com/pub/Collateral/MMBZ5V6ALT1-D.PDF" (id 3) (at 120.65 97.79 90)
+      (effects (font (size 1.27 1.27)) hide)
+    )
+    (property "Part Number" "MMBZ5V6ALFHT116" (id 4) (at 123.19 97.79 0)
+      (effects (font (size 1.27 1.27)) hide)
+    )
+    (pin "1")
+    (pin "2")
+    (pin "3")
+  )
   (symbol (lib_id "Device:C_Small") (at 224.79 50.8 0) (unit 1)
     (in_bom yes) (on_board yes) (fields_autoplaced)
@@
     (pin "1")
   )
+  (symbol (lib_id "power:GND") (at 123.19 140.97 0) (unit 1)
+    (in_bom yes) (on_board yes) (fields_autoplaced)
+    (property "Reference" "#PWR0113" (id 0) (at 123.19 147.32 0)
+      (effects (font (size 1.27 1.27)) hide)
+    )
+    (property "Value" "GND" (id 1) (at 123.19 146.05 0))
+    (property "Footprint" "" (id 2) (at 123.19 140.97 0)
+      (effects (font (size 1.27 1.27)) hide)
+    )
+    (property "Datasheet" "" (id 3) (at 123.19 140.97 0)
+      (effects (font (size 1.27 1.27)) hide)
+    )
+    (pin "1")
+  )
   (symbol (lib_id "Device:R_Small") (at 157.48 120.65 270) (mirror x) (unit 1)
     (in_bom yes) (on_board yes)
@@
       (reference "#PWR0112") (unit 1) (value "GND") (footprint "")
     )
+    (path "/b08a5218-3c22-4695-ab71-ac0793f0ef12"
+      (reference "#PWR0113") (unit 1) (value "GND") (footprint "")
+    )
     (path "/1b1ae3dd-f20e-4dc4-843b-d424ca135075/0056e9b6-9e95-45b5-baf9-a3f1f3b0cfb6"
       (reference "C1") (unit 1) (value "4.7u") (footprint "Capacitor_SMD:C_0805_2012Metric")
@@
       (reference "D2") (unit 1) (value "Red") (footprint "LED_SMD:LED_1206_3216Metric")
     )
+    (path "/5cd8fe45-fa49-4729-81c8-b7c257fc3660"
+      (reference "D3") (unit 1) (value "MMBZxx") (footprint "Package_TO_SOT_SMD:SOT-23")
+    )
     (path "/1b1ae3dd-f20e-4dc4-843b-d424ca135075/3f6b5f2a-45d9-4080-aba4-0ff576a8a80f"

Commit message: finished pcb
Parts:
- removed SW1: SW_DIP_x02, DS04-254-2-02BK-SMT:SW_DS04-254-2-02BK-SMT, symbol Switch:SW_DIP_x02
- added JP2, JP3: Jumper_2_Open, Jumper:SolderJumper-2_P1.3mm_Open_RoundedPad1.0x1.5mm, symbol Jumper:Jumper_2_Open
- added TP4, TP5: TestPoint_Small, TestPoint:TestPoint_Loop_D2.54mm_Drill1.5mm_Beaded, symbol Connector:TestPoint_Small
Connections:
- net DCNF0: now also JP2.2 (B)
- net DCNF1: now also JP3.2 (B)
- net GND: now also TP5.1
- net VBUS: now also TP4.1
- net VCCIO: now also JP2.1 (A), JP3.1 (A)
Changed lines of the file:
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@@
   (junction (at 194.31 125.73) (diameter 0) (color 0 0 0 0)
   )
+  (junction (at 76.2 124.46) (diameter 0) (color 0 0 0 0)
+  )
   (junction (at 151.13 120.65) (diameter 0) (color 0 0 0 0)
   )
@@
   )
   (junction (at 114.3 43.18) (diameter 0) (color 0 0 0 0)
+  )
+  (junction (at 92.71 72.39) (diameter 0) (color 0 0 0 0)
   )
   (junction (at 125.73 83.82) (diameter 0) (color 0 0 0 0)
@@
     (stroke (width 0) (type default))
   )
-  (wire (pts (xy 109.22 45.72) (xy 121.92 45.72))
+  (wire (pts (xy 106.68 45.72) (xy 121.92 45.72))
     (stroke (width 0) (type default))
   )
@@
     (stroke (width 0) (type default))
   )
-  (wire (pts (xy 76.2 110.49) (xy 76.2 140.97))
+  (wire (pts (xy 76.2 110.49) (xy 76.2 124.46))
     (stroke (width 0) (type default))
   )
@@
     (stroke (width 0) (type default))
   )
+  (wire (pts (xy 92.71 72.39) (xy 93.98 72.39))
+    (stroke (width 0) (type default))
+  )
   (wire (pts (xy 162.56 68.58) (xy 162.56 102.87))
     (stroke (width 0) (type default))
@@
     (stroke (width 0) (type default))
   )
-  (wire (pts (xy 109.22 43.18) (xy 114.3 43.18))
+  (wire (pts (xy 106.68 43.18) (xy 114.3 43.18))
     (stroke (width 0) (type default))
   )
@@
     (stroke (width 0) (type default))
   )
+  (wire (pts (xy 91.44 72.39) (xy 92.71 72.39))
+    (stroke (width 0) (type default))
+  )
   (wire (pts (xy 163.83 119.38) (xy 163.83 120.65))
     (stroke (width 0) (type default))
@@
     (stroke (width 0) (type default))
   )
-  (wire (pts (xy 93.98 45.72) (xy 91.44 45.72))
+  (wire (pts (xy 91.44 45.72) (xy 96.52 45.72))
     (stroke (width 0) (type default))
   )
@@
     (stroke (width 0) (type default))
   )
+  (wire (pts (xy 76.2 124.46) (xy 76.2 140.97))
+    (stroke (width 0) (type default))
+  )
   (wire (pts (xy 215.9 45.72) (xy 215.9 46.99))
     (stroke (width 0) (type default))
@@
     (stroke (width 0) (type default))
   )
-  (wire (pts (xy 91.44 43.18) (xy 93.98 43.18))
+  (wire (pts (xy 91.44 43.18) (xy 96.52 43.18))
     (stroke (width 0) (type default))
   )
@@
     )
   )
-  (global_label "VBUS" (shape input) (at 91.44 72.39 0) (fields_autoplaced)
+  (global_label "VBUS" (shape input) (at 93.98 72.39 0) (fields_autoplaced)
     (effects (font (size 1.27 1.27)) (justify left))
-    (property "Intersheet References" "${INTERSHEET_REFS}" (id 0) (at 98.7517 72.3106 0)
+    (property "Intersheet References" "${INTERSHEET_REFS}" (id 0) (at 101.2917 72.3106 0)
       (effects (font (size 1.27 1.27)) (justify left))
     )
@@
     (pin "2")
   )
+  (symbol (lib_id "Jumper:Jumper_2_Open") (at 101.6 45.72 0) (mirror x) (unit 1)
+    (in_bom yes) (on_board yes)
+    (property "Reference" "JP3" (id 0) (at 101.6 49.53 0)
+      (effects (font (size 1.27 1.27)))
+    )
+    (property "Value" "Jumper_2_Open" (id 1) (at 101.6 48.26 0)
+      (effects (font (size 1.27 1.27)) hide)
+    )
+    (property "Footprint" "Jumper:SolderJumper-2_P1.3mm_Open_RoundedPad1.0x1.5mm" (id 2) (at 101.6 45.72 0)
+      (effects (font (size 1.27 1.27)) hide)
+    )
+    (property "Datasheet" "~" (id 3) (at 101.6 45.72 0)
+      (effects (font (size 1.27 1.27)) hide)
+    )
+    (pin "1")
+    (pin "2")
+  )
   (symbol (lib_id "power:GND") (at 143.51 140.97 0) (unit 1)
     (in_bom yes) (on_board yes) (fields_autoplaced)
@@
     (pin "1")
     (pin "2")
-  )
-  (symbol (lib_id "Switch:SW_DIP_x02") (at 101.6 45.72 0) (unit 1)
-    (in_bom yes) (on_board yes) (fields_autoplaced)
-    (property "Reference" "SW1" (id 0) (at 101.6 35.56 0)
-      (effects (font (size 1.27 1.27)))
-    )
-    (property "Value" "SW_DIP_x02" (id 1) (at 101.6 38.1 0)
-      (effects (font (size 1.27 1.27)))
-    )
-    (property "Footprint" "DS04-254-2-02BK-SMT:SW_DS04-254-2-02BK-SMT" (id 2) (at 101.6 45.72 0)
-      (effects (font (size 1.27 1.27)) hide)
-    )
-    (property "Datasheet" "~" (id 3) (at 101.6 45.72 0)
-      (effects (font (size 1.27 1.27)) hide)
-    )
-    (property "Part Number" "DS04-254-2-02BK-SMT" (id 4) (at 101.6 45.72 0)
-      (effects (font (size 1.27 1.27)) hide)
-    )
-    (pin "1")
-    (pin "2")
-    (pin "3")
-    (pin "4")
   )
   (symbol (lib_id "Device:R_Small") (at 96.52 106.68 0) (unit 1)
@@
       (effects (font (size 1.27 1.27)) hide)
     )
+  )
+  (symbol (lib_id "Connector:TestPoint_Small") (at 92.71 72.39 0) (unit 1)
+    (in_bom yes) (on_board yes)
+    (property "Reference" "TP4" (id 0) (at 91.44 69.85 0)
+      (effects (font (size 1.27 1.27)) (justify left))
+    )
+    (property "Value" "TestPoint_Small" (id 1) (at 93.98 74.295 0)
+      (effects (font (size 1.27 1.27)) (justify left) hide)
+    )
+    (property "Footprint" "TestPoint:TestPoint_Loop_D2.54mm_Drill1.5mm_Beaded" (id 2) (at 97.79 72.39 0)
+      (effects (font (size 1.27 1.27)) hide)
+    )
+    (property "Datasheet" "~" (id 3) (at 97.79 72.39 0)
+      (effects (font (size 1.27 1.27)) hide)
+    )
+    (pin "1")
   )
   (symbol (lib_id "Mechanical:MountingHole") (at 57.15 231.14 0) (unit 1)
@@
     (pin "S1")
   )
+  (symbol (lib_id "Jumper:Jumper_2_Open") (at 101.6 43.18 0) (unit 1)
+    (in_bom yes) (on_board yes) (fields_autoplaced)
+    (property "Reference" "JP2" (id 0) (at 101.6 40.64 0)
+      (effects (font (size 1.27 1.27)))
+    )
+    (property "Value" "Jumper_2_Open" (id 1) (at 101.6 40.64 0)
+      (effects (font (size 1.27 1.27)) hide)
+    )
+    (property "Footprint" "Jumper:SolderJumper-2_P1.3mm_Open_RoundedPad1.0x1.5mm" (id 2) (at 101.6 43.18 0)
+      (effects (font (size 1.27 1.27)) hide)
+    )
+    (property "Datasheet" "~" (id 3) (at 101.6 43.18 0)
+      (effects (font (size 1.27 1.27)) hide)
+    )
+    (pin "1")
+    (pin "2")
+  )
   (symbol (lib_id "Device:R_Small") (at 135.89 77.47 0) (unit 1)
     (in_bom yes) (on_board yes)
@@
     (pin "1")
     (pin "2")
+  )
+  (symbol (lib_id "Connector:TestPoint_Small") (at 76.2 124.46 0) (unit 1)
+    (in_bom yes) (on_board yes)
+    (property "Reference" "TP5" (id 0) (at 71.12 124.46 0)
+      (effects (font (size 1.27 1.27)) (justify left))
+    )
+    (property "Value" "TestPoint_Small" (id 1) (at 77.47 126.365 0)
+      (effects (font (size 1.27 1.27)) (justify left) hide)
+    )
+    (property "Footprint" "TestPoint:TestPoint_Loop_D2.54mm_Drill1.5mm_Beaded" (id 2) (at 81.28 124.46 0)
+      (effects (font (size 1.27 1.27)) hide)
+    )
+    (property "Datasheet" "~" (id 3) (at 81.28 124.46 0)
+      (effects (font (size 1.27 1.27)) hide)
+    )
+    (pin "1")
   )
   (symbol (lib_id "Device:C_Small") (at 151.13 135.89 0) (mirror y) (unit 1)
@@
       (reference "JP1") (unit 1) (value "Jumper_2_Bridged") (footprint "Jumper:SolderJumper-2_P1.3mm_Bridged_RoundedPad1.0x1.5mm")
     )
+    (path "/93d2313f-0919-4c6f-b07d-ab630442d056"
+      (reference "JP2") (unit 1) (value "Jumper_2_Open") (footprint "Jumper:SolderJumper-2_P1.3mm_Open_RoundedPad1.0x1.5mm")
+    )
+    (path "/48e8d634-1608-4cd1-814c-418fcd84837c"
+      (reference "JP3") (unit 1) (value "Jumper_2_Open") (footprint "Jumper:SolderJumper-2_P1.3mm_Open_RoundedPad1.0x1.5mm")
+    )
     (path "/1b1ae3dd-f20e-4dc4-843b-d424ca135075/308e38e3-4b9c-4dc0-a69a-03805e5e5354"
       (reference "Q1") (unit 1) (value "Q_PNP_BCE") (footprint "Package_TO_SOT_SMD:SOT-23")
@@
       (reference "R22") (unit 1) (value "220") (footprint "Resistor_SMD:R_0603_1608Metric")
     )
-    (path "/68dd0864-7308-416d-96e0-57c47ec6c321"
-      (reference "SW1") (unit 1) (value "SW_DIP_x02") (footprint "DS04-254-2-02BK-SMT:SW_DS04-254-2-02BK-SMT")
-    )
     (path "/4f926a51-5226-43cc-9957-25202b8286cb/cdcbcf86-ac45-44c4-b214-16377dfbc45b"
       (reference "SW2") (unit 1) (value "Reset") (footprint "Button_Switch_SMD:Panasonic_EVQPUJ_EVQPUA")
     )
+    (path "/1b1ae3dd-f20e-4dc4-843b-d424ca135075/5e14c1a8-7e4d-4106-9180-6229f7fc13aa"
+      (reference "TP1") (unit 1) (value "TestPoint_Small") (footprint "TestPoint:TestPoint_Loop_D2.54mm_Drill1.5mm_Beaded")
+    )
+    (path "/1b1ae3dd-f20e-4dc4-843b-d424ca135075/321ab144-417b-431f-b921-19f51870b74c"
+      (reference "TP2") (unit 1) (value "TestPoint_Small") (footprint "TestPoint:TestPoint_Loop_D2.54mm_Drill1.5mm_Beaded")
+    )
+    (path "/1b1ae3dd-f20e-4dc4-843b-d424ca135075/e888e497-49a1-4762-a080-601d074dad4a"
+      (reference "TP3") (unit 1) (value "TestPoint_Small") (footprint "TestPoint:TestPoint_Loop_D2.54mm_Drill1.5mm_Beaded")
+    )
+    (path "/6ee2eff6-d2ee-43b3-a39c-023a759b20f4"
+      (reference "TP4") (unit 1) (value "TestPoint_Small") (footprint "TestPoint:TestPoint_Loop_D2.54mm_Drill1.5mm_Beaded")
+    )
+    (path "/c499d360-d3af-4d45-a462-1acb7527a42f"
+      (reference "TP5") (unit 1) (value "TestPoint_Small") (footprint "TestPoint:TestPoint_Loop_D2.54mm_Drill1.5mm_Beaded")
+    )
     (path "/1b1ae3dd-f20e-4dc4-843b-d424ca135075/c13225c4-79d5-46c5-bda7-8b930472369d"
