File: pcb/schematics/bus.kicad_sch (KiCad schematic)
At the start: 1 part, among them J1 09032967825

Commit message: finished the board
Other:
- title: (none) -> Bus
Changed lines of the file:
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@@
 (kicad_sch (version 20220126) (generator eeschema)
   (paper "A4")
+  (title_block
+    (title "Bus")
+    (date "2022-02-26")
+    (rev "1.0")
+  )
   (junction (at 143.51 168.91) (diameter 0) (color 0 0 0 0)
   )
