File: pcb/schematics/mcu.kicad_sch (KiCad schematic)
At the start: 25 parts, among them J3 Conn_01x06_Female, SW2 Reset, U3 STM32F103V8Tx, Y2 24MHz

Commit message: finished pcb
Connections:
- no-connect marks 0 -> 17
Changed lines of the file:
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@@
   (junction (at 87.63 35.56) (diameter 0) (color 0 0 0 0)
   )
+  (no_connect (at 172.72 46.99))
+  (no_connect (at 172.72 49.53))
+  (no_connect (at 172.72 52.07))
+  (no_connect (at 172.72 54.61))
+  (no_connect (at 172.72 92.71))
+  (no_connect (at 172.72 133.35))
+  (no_connect (at 172.72 135.89))
+  (no_connect (at 172.72 138.43))
+  (no_connect (at 172.72 140.97))
+  (no_connect (at 172.72 166.37))
+  (no_connect (at 172.72 168.91))
+  (no_connect (at 172.72 171.45))
+  (no_connect (at 121.92 97.79))
+  (no_connect (at 121.92 95.25))
+  (no_connect (at 121.92 100.33))
+  (no_connect (at 121.92 102.87))
+  (no_connect (at 121.92 105.41))
   (wire (pts (xy 167.64 27.94) (xy 171.45 27.94))
     (stroke (width 0) (type default))

Commit message: finished the board
Other:
- title: (none) -> MCU
Changed lines of the file:
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@@
 (kicad_sch (version 20220126) (generator eeschema)
   (paper "A4")
+  (title_block
+    (title "MCU")
+    (date "2022-02-26")
+    (rev "1.0")
+  )
   (junction (at 154.94 27.94) (diameter 0) (color 0 0 0 0)
   )
