File: pcb/schematics/power.kicad_sch (KiCad schematic)
At the start: 21 parts, among them Q1 Q_PNP_BCE, U1 STLQ020PU33R

Commit message: finish the schematic
Parts:
- removed Q1, Q?: Q_PNP_BCE, symbol Device:Q_PNP_BCE
- removed R1: 10k, symbol Device:R_Small
- removed R2: R_Small, symbol Device:R_Small
- added C27: 100n, Capacitor_SMD:C_0603_1608Metric, symbol Device:C_Small
- added JP1: Jumper_2_Bridged, Jumper:SolderJumper-2_P1.3mm_Bridged_RoundedPad1.0x1.5mm, symbol Jumper:Jumper_2_Bridged
- added R14: 10k, Resistor_SMD:R_0603_1608Metric, symbol Device:R_Small
- added R15: 68k, Resistor_SMD:R_0603_1608Metric, symbol Device:R_Small
- added U5: SN74ALVC00, Package_SO:TSSOP-14_4.4x5mm_P0.65mm, symbol SN74ALVC00:SN74ALVC00
- added U6: MIC94090, Package_TO_SOT_SMD:SOT-363_SC-70-6, symbol MIC94090:MIC94090
- D1: renamed from D?; footprint (none) -> LED_SMD:LED_1206_3216Metric; Part Number (none) -> 156120VS75300
- D2: renamed from D?; footprint (none) -> LED_SMD:LED_1206_3216Metric; Part Number (none) -> 156120RS75300
- FB1: footprint (none) -> Inductor_SMD:L_1206_3216Metric; Part Number (none) -> MH3261-601Y
- Q1: renamed from Q?; footprint (none) -> Package_TO_SOT_SMD:SOT-23; symbol Device:Q_PNP_BCE -> Device:Q_PNP_BEC; Part Number (none) -> BC857,215
- R1: renamed from R?; value R_Small -> 160mOhm; footprint (none) -> Resistor_SMD:R_0805_2012Metric; Part Number (none) -> RL1220S-R16-F
- R16: renamed from R?; value 220 -> 374; footprint (none) -> Resistor_SMD:R_0603_1608Metric; Part Number (none) -> CR0603-FX-3740ELF
- R17: renamed from R?; footprint (none) -> Resistor_SMD:R_0603_1608Metric; Part Number (none) -> RC0603FR-07220RL
- R2: renamed from R?; footprint (none) -> Resistor_SMD:R_0603_1608Metric; Part Number (none) -> CR0603-FX-1002ELF
- U4: renamed from U?; footprint (none) -> Package_SO:VSSOP-10_3x3mm_P0.5mm; Part Number (none) -> INA381A1IDGSR
- gave numbers to parts that had none: 1
Connections:
- net +3V3: now also Q1.2 (E), C27.1, R14.1, U5.14 (Vcc); no longer Q1.3 (E)
- net +5V: now also U6.4 (Vin)
- net +5V_Mod: now also U6.1 (Vout)
- net GND: now also C27.2, R15.2, U5.7 (GND), U6.2 (GND), U6.5 (GND)
- net MODULE_ENABLE: now also U5.1 (1A)
- net at D2.2 (A): now also Q1.3 (C), JP1.1 (A); no longer Q1.2 (C)
- net at U4.7 (CMPREF): now also R14.2, R15.1
- net RESET renamed MODULE_RESET
- new net: U5.10 (3B), U5.3 (1Y), U5.9 (3A)
- new net: U5.8 (3Y), U6.6 (EN)
- new net: U5.2 (1B), U5.6 (2Y)
- new net OVERCURRENT_SENSE: JP1.2 (B), U5.4 (2A), U5.5 (2B)
Other:
- note added: "0"
- note added: "1"
- note added: "Imax = 1A Pd_max = 250mW Rsense_max = Pd_max / Imax^2 = 250mOhm With G=20V/V, R = 160mOhm -> V at 1A = 3.2V"
- note added: "MODULE_ENABLE"
- note added: "OUTPUT_ENABLE"
- note added: "OVERCURRENT_SENSE"
- note added: "V = 3.2V -> I = 1A V = 2.88 -> I = 900mA R1 = 10k and R2 = 68k"
- note removed: "INA381 to shutdown module if USB power is too big"
- note removed: "MODULE_ENABLE should be connected to an open-drain output"
- moved on the sheet: C1, C2, C28, C3, C4, C5, D1, D2, FB1, Q1, R1, R16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

Commit message: finished pcb
Parts:
- added TP1, TP2, TP3: TestPoint_Small, TestPoint:TestPoint_Loop_D2.54mm_Drill1.5mm_Beaded, symbol Connector:TestPoint_Small
Connections:
- net +3V3: now also TP1.1
- net +5V_Mod: now also TP2.1
- net CURRENT_SENSE: now also TP3.1
Changed lines of the file:
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@@
   (junction (at 248.92 139.7) (diameter 0) (color 0 0 0 0)
   )
+  (junction (at 86.36 143.51) (diameter 0) (color 0 0 0 0)
+  )
   (junction (at 171.45 147.32) (diameter 0) (color 0 0 0 0)
   )
@@
   (junction (at 62.23 55.88) (diameter 0) (color 0 0 0 0)
   )
+  (junction (at 252.73 139.7) (diameter 0) (color 0 0 0 0)
+  )
   (junction (at 191.77 55.88) (diameter 0) (color 0 0 0 0)
   )
@@
   (junction (at 52.07 124.46) (diameter 0) (color 0 0 0 0)
   )
+  (junction (at 231.14 55.88) (diameter 0) (color 0 0 0 0)
+  )
   (junction (at 87.63 140.97) (diameter 0) (color 0 0 0 0)
   )
@@
     (stroke (width 0) (type default))
   )
+  (wire (pts (xy 86.36 143.51) (xy 88.9 143.51))
+    (stroke (width 0) (type default))
+  )
   (wire (pts (xy 52.07 123.19) (xy 52.07 124.46))
     (stroke (width 0) (type default))
@@
     (stroke (width 0) (type default))
   )
+  (wire (pts (xy 252.73 139.7) (xy 255.27 139.7))
+    (stroke (width 0) (type default))
+  )
   (wire (pts (xy 194.31 58.42) (xy 191.77 58.42))
     (stroke (width 0) (type default))
@@
     (stroke (width 0) (type default))
   )
-  (wire (pts (xy 248.92 139.7) (xy 255.27 139.7))
-    (stroke (width 0) (type default))
-  )
-  (wire (pts (xy 231.14 55.88) (xy 226.06 55.88))
+  (wire (pts (xy 248.92 139.7) (xy 252.73 139.7))
+    (stroke (width 0) (type default))
+  )
+  (wire (pts (xy 226.06 55.88) (xy 231.14 55.88))
     (stroke (width 0) (type default))
   )
@@
     (effects (font (size 1.27 1.27)) (justify right bottom))
   )
-  (global_label "CURRENT_SENSE" (shape input) (at 86.36 143.51 0) (fields_autoplaced)
+  (global_label "CURRENT_SENSE" (shape input) (at 88.9 143.51 0) (fields_autoplaced)
     (effects (font (size 1.27 1.27)) (justify left))
-    (property "Intersheet References" "${INTERSHEET_REFS}" (id 0) (at 104.376 143.4306 0)
+    (property "Intersheet References" "${INTERSHEET_REFS}" (id 0) (at 106.916 143.4306 0)
       (effects (font (size 1.27 1.27)) (justify left))
     )
@@
     (pin "2")
   )
+  (symbol (lib_id "Connector:TestPoint_Small") (at 252.73 139.7 0) (unit 1)
+    (in_bom yes) (on_board yes)
+    (property "Reference" "TP2" (id 0) (at 251.46 137.16 0)
+      (effects (font (size 1.27 1.27)) (justify left))
+    )
+    (property "Value" "TestPoint_Small" (id 1) (at 254 141.605 0)
+      (effects (font (size 1.27 1.27)) (justify left) hide)
+    )
+    (property "Footprint" "TestPoint:TestPoint_Loop_D2.54mm_Drill1.5mm_Beaded" (id 2) (at 257.81 139.7 0)
+      (effects (font (size 1.27 1.27)) hide)
+    )
+    (property "Datasheet" "~" (id 3) (at 257.81 139.7 0)
+      (effects (font (size 1.27 1.27)) hide)
+    )
+    (pin "1")
+  )
   (symbol (lib_id "Device:FerriteBead_Small") (at 100.33 55.88 90) (unit 1)
     (in_bom yes) (on_board yes) (fields_autoplaced)
@@
     (pin "2")
     (pin "3")
+  )
+  (symbol (lib_id "Connector:TestPoint_Small") (at 231.14 55.88 0) (unit 1)
+    (in_bom yes) (on_board yes)
+    (property "Reference" "TP1" (id 0) (at 232.41 55.88 0)
+      (effects (font (size 1.27 1.27)) (justify left))
+    )
+    (property "Value" "TestPoint_Small" (id 1) (at 232.41 57.785 0)
+      (effects (font (size 1.27 1.27)) (justify left) hide)
+    )
+    (property "Footprint" "TestPoint:TestPoint_Loop_D2.54mm_Drill1.5mm_Beaded" (id 2) (at 236.22 55.88 0)
+      (effects (font (size 1.27 1.27)) hide)
+    )
+    (property "Datasheet" "~" (id 3) (at 236.22 55.88 0)
+      (effects (font (size 1.27 1.27)) hide)
+    )
+    (pin "1")
   )
   (symbol (lib_id "power:+3V3") (at 34.29 123.19 0) (unit 1)
@@
     (pin "2")
   )
+  (symbol (lib_id "Connector:TestPoint_Small") (at 86.36 143.51 0) (unit 1)
+    (in_bom yes) (on_board yes)
+    (property "Reference" "TP3" (id 0) (at 85.09 146.05 0)
+      (effects (font (size 1.27 1.27)) (justify left))
+    )
+    (property "Value" "TestPoint_Small" (id 1) (at 87.63 145.415 0)
+      (effects (font (size 1.27 1.27)) (justify left) hide)
+    )
+    (property "Footprint" "TestPoint:TestPoint_Loop_D2.54mm_Drill1.5mm_Beaded" (id 2) (at 91.44 143.51 0)
+      (effects (font (size 1.27 1.27)) hide)
+    )
+    (property "Datasheet" "~" (id 3) (at 91.44 143.51 0)
+      (effects (font (size 1.27 1.27)) hide)
+    )
+    (pin "1")
+  )
   (symbol (lib_id "power:+3V3") (at 121.92 123.19 0) (unit 1)

Commit message: finished the board
Other:
- title: (none) -> Power
Changed lines of the file:
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@@
 (kicad_sch (version 20220126) (generator eeschema)
   (paper "A4")
+  (title_block
+    (title "Power")
+    (date "2022-02-26")
+    (rev "1.0")
+  )
   (junction (at 81.28 55.88) (diameter 0) (color 0 0 0 0)
   )
